File: FT230X Breakout.brd (EAGLE design)
At the start: 54.6 x 32.7 mm, 20 parts, among them U1 FT230XSSOP

Commit message: Updated Files
Updated file names. Added PDF version of schematic. Changed frame in
file.
Parts:
- removed FRAME1: FRAME-LETTER, SparkFun-Aesthetics:CREATIVE_COMMONS
Changed lines of the file:
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@@
 </autorouter>
 <elements>
-<element name="FRAME1" library="SparkFun-Aesthetics" package="CREATIVE_COMMONS" value="FRAME-LETTER" x="5.08" y="-7.62"/>
 <element name="JP1" library="SparkFun-Connectors" package="1X07" value="" x="46.99" y="24.13" rot="R270"/>
 <element name="JP2" library="SparkFun-Connectors" package="USB-MINIB" value="USBSMD" x="5.08" y="15.24"/>
